Commit message: implemented inverse kinematics for robotic arm control and fixing the gap in the robot

File: uf850_description/urdf/uf850.urdf (robot description, URDF)
Before this commit: robot uf850, 7 links, 6 joints
Links:
- added link camera_link, mass 0.05; visual box size=0.05 0.05 0.05
Joints:
- added joint camera_mount_joint: type fixed, parent link6, child camera_link, origin xyz=0 0 0 rpy=0 0 0
- joint base_to_link1: origin xyz=0 0 0.2 rpy=0 0 0 -> xyz=0 0 0.15 rpy=0 0 0
- joint link3_to_link4: origin xyz=0.15 -0.15 0 rpy=1.57 0 0 -> xyz=0.1 -0.15 0 rpy=1.57 0 0
